Commit message: Fix segmentation fault: initialize UKF and LiDAR subscribers, fix LiDAR mesh paths

File: bluerov2_description/urdf/sensors.xacro (robot description, xacro)
@@ -49,5 +49,5 @@
     <visual>
       <geometry>
-        <mesh filename="https://app.gazebosim.org/OpenRobotics/fuel/models/Lidar%202d%20v1" scale="1 1 1"/>
+        <mesh filename="file://$(find bluerov2_description)/meshes/lidar.dae" scale="1 1 1"/>
       </geometry>
     </visual>
@@ -71,5 +71,5 @@
     <visual>
       <geometry>
-        <mesh filename="https://app.gazebosim.org/OpenRobotics/fuel/models/Lidar%202d%20v1" scale="1 1 1"/>
+        <mesh filename="file://$(find bluerov2_description)/meshes/lidar.dae" scale="1 1 1"/>
       </geometry>
     </visual>
@@ -93,5 +93,5 @@
     <visual>
       <geometry>
-        <mesh filename="https://app.gazebosim.org/OpenRobotics/fuel/models/Lidar%202d%20v1" scale="1 1 1"/>
+        <mesh filename="file://$(find bluerov2_description)/meshes/lidar.dae" scale="1 1 1"/>
       </geometry>
     </visual>

Commit message: Use downloaded LiDAR model from Gazebo Fuel for visual representation

File: bluerov2_description/urdf/sensors.xacro (robot description, xacro)
@@ -44,10 +44,10 @@
     range_max="20.0"
     range_stddev="0.01"
-    mesh="file://$(find bluerov2_description)/meshes/lidar.dae">
+    mesh="file://$(find bluerov2_description)/meshes/ping1d.dae">
     <inertia ixx="0.00001" ixy="0.0" ixz="0.0" iyy="0.00001" iyz="0.0" izz="0.00001" />
     <origin xyz="0 0.15 0" rpy="0 0 1.5708"/>
     <visual>
       <geometry>
-        <mesh filename="file://$(find bluerov2_description)/meshes/lidar.dae" scale="1 1 1"/>
+        <mesh filename="file://$(find bluerov2_description)/../Lidar/meshes/lidar_2d_v1.dae" scale="1 1 1"/>
       </geometry>
     </visual>
@@ -66,10 +66,10 @@
     range_max="20.0"
     range_stddev="0.01"
-    mesh="file://$(find bluerov2_description)/meshes/lidar.dae">
+    mesh="file://$(find bluerov2_description)/meshes/ping1d.dae">
     <inertia ixx="0.00001" ixy="0.0" ixz="0.0" iyy="0.00001" iyz="0.0" izz="0.00001" />
     <origin xyz="0 -0.15 0" rpy="0 0 -1.5708"/>
     <visual>
       <geometry>
-        <mesh filename="file://$(find bluerov2_description)/meshes/lidar.dae" scale="1 1 1"/>
+        <mesh filename="file://$(find bluerov2_description)/../Lidar/meshes/lidar_2d_v1.dae" scale="1 1 1"/>
       </geometry>
     </visual>
@@ -88,10 +88,10 @@
     range_max="20.0"
     range_stddev="0.01"
-    mesh="file://$(find bluerov2_description)/meshes/lidar.dae">
+    mesh="file://$(find bluerov2_description)/meshes/ping1d.dae">
     <inertia ixx="0.00001" ixy="0.0" ixz="0.0" iyy="0.00001" iyz="0.0" izz="0.00001" />
     <origin xyz="0.2 0 0" rpy="0 0 0"/>
     <visual>
       <geometry>
-        <mesh filename="file://$(find bluerov2_description)/meshes/lidar.dae" scale="1 1 1"/>
+        <mesh filename="file://$(find bluerov2_description)/../Lidar/meshes/lidar_2d_v1.dae" scale="1 1 1"/>
       </geometry>
     </visual>

Commit message: Fix ACADOS QP solver issues and optimize LiDAR configuration for straight line navigation

File: bluerov2_description/urdf/sensors.xacro (robot description, xacro)
@@ -31,49 +31,5 @@
   <xacro:default_gps namespace="${namespace}" parent_link="${namespace}/base_link" />
   <!-- Mount LiDAR sensors for straight line navigation -->
-  <!-- Left side LiDAR -->
-  <xacro:bluerov2_sss
-    namespace="${namespace}"
-    parent_link="${namespace}/base_link"
-    topic="left_lidar_"
-    suffix="left"
-    mass="0.001"
-    update_rate="20"
-    samples="180"
-    fov="3.14"
-    range_min="0.1"
-    range_max="20.0"
-    range_stddev="0.01"
-    mesh="file://$(find bluerov2_description)/meshes/ping1d.dae">
-    <inertia ixx="0.00001" ixy="0.0" ixz="0.0" iyy="0.00001" iyz="0.0" izz="0.00001" />
-    <origin xyz="0 0.15 0" rpy="0 0 1.5708"/>
-    <visual>
-      <geometry>
-        <mesh filename="file://$(find bluerov2_description)/../Lidar/meshes/lidar_2d_v1.dae" scale="1 1 1"/>
-      </geometry>
-    </visual>
-  </xacro:bluerov2_sss>
-  <!-- Right side LiDAR -->
-  <xacro:bluerov2_sss
-    namespace="${namespace}"
-    parent_link="${namespace}/base_link"
-    topic="right_lidar_"
-    suffix="right"
-    mass="0.001"
-    update_rate="20"
-    samples="180"
-    fov="3.14"
-    range_min="0.1"
-    range_max="20.0"
-    range_stddev="0.01"
-    mesh="file://$(find bluerov2_description)/meshes/ping1d.dae">
-    <inertia ixx="0.00001" ixy="0.0" ixz="0.0" iyy="0.00001" iyz="0.0" izz="0.00001" />
-    <origin xyz="0 -0.15 0" rpy="0 0 -1.5708"/>
-    <visual>
-      <geometry>
-        <mesh filename="file://$(find bluerov2_description)/../Lidar/meshes/lidar_2d_v1.dae" scale="1 1 1"/>
-      </geometry>
-    </visual>
-  </xacro:bluerov2_sss>
-  <!-- Forward LiDAR for obstacle detection -->
+  <!-- Forward LiDAR for obstacle detection and navigation -->
   <xacro:bluerov2_sss
     namespace="${namespace}"

Commit message: Add LiDAR laser visualization in RViz
- Enhanced LiDAR sensor configuration with laser visualization
- Created dedicated RViz config for LiDAR display
- Added material file for LiDAR visual effects
- Created LiDAR test script and launch file
- Modified main launch file to use LiDAR RViz config
- Added visualize_rays and always_on parameters
- Enhanced laser intensity and color settings

File: bluerov2_description/urdf/sensors.xacro (robot description, xacro)
@@ -51,4 +51,5 @@
         <mesh filename="file://$(find bluerov2_description)/../Lidar/meshes/lidar_2d_v1.dae" scale="1 1 1"/>
       </geometry>
+      <material name="lidar_material"/>
     </visual>
   </xacro:bluerov2_sss>

File: bluerov2_description/urdf/snippets.xacro (robot description, xacro)
@@ -208,7 +208,12 @@
         </noise>
       </ray>
+      <!-- Enhanced visualization for LiDAR laser -->
+      <visualize_rays>true</visualize_rays>
+      <always_on>true</always_on>
       <plugin name="sonar${suffix}_controller" filename="libgazebo_ros_laser.so">
         <topicName>${topic}${suffix}</topicName>
         <frameName>sonar${suffix}_link</frameName>
+        <minIntensity>0.1</minIntensity>
+        <maxIntensity>1.0</maxIntensity>
       </plugin>
     </sensor>
